Commit message: fix xbot urdf

File: jbot_description/urdf/xbot_urdf.urdf (robot description, URDF)
Before this commit: robot xbot_urdf, 6 links, 5 joints
Joints:
- joint joint_2: axis 1 0 0 -> -1 0 0
- joint joint_4: axis 1 0 0 -> -1 0 0

File: jbot_description/urdf/xbot_urdf_left.urdf (robot description, URDF)
Before this commit: robot xbot_urdf, 6 links, 5 joints
Joints:
- joint joint_21: axis 1 0 0 -> -1 0 0
- joint joint_41: axis 1 0 0 -> -1 0 0
